Commit message: fr3: Franka fr3v2 visual meshes, one STL per colour with its URDF material, in place of the colourless STLs

File: assets/urdf/fr3_xhand_description/fr3_xhand/fr3_xhand.urdf (robot description, URDF)
Before this commit: robot fr3_xhand, 39 links, 38 joints
Links:
- link fr3_link0: geometry collision mesh filename=../fr3/meshes/collision/link0.stl; visual mesh filename=../fr3/meshes/visual/link0_0.stl
- link fr3_link1: geometry collision mesh filename=../fr3/meshes/collision/link1.stl; visual mesh filename=../fr3/meshes/visual/link1_0.stl
- link fr3_link2: geometry collision mesh filename=../fr3/meshes/collision/link2.stl; visual mesh filename=../fr3/meshes/visual/link2_0.stl
- link fr3_link3: geometry collision mesh filename=../fr3/meshes/collision/link3.stl; visual mesh filename=../fr3/meshes/visual/link3_0.stl
- link fr3_link4: geometry collision mesh filename=../fr3/meshes/collision/link4.stl; visual mesh filename=../fr3/meshes/visual/link4_0.stl
- link fr3_link5: geometry collision mesh filename=../fr3/meshes/collision/link5.stl; visual mesh filename=../fr3/meshes/visual/link5_0.stl
- link fr3_link6: geometry collision mesh filename=../fr3/meshes/collision/link6.stl; visual mesh filename=../fr3/meshes/visual/link6_0.stl
- link fr3_link7: geometry collision mesh filename=../fr3/meshes/collision/link7.stl; visual mesh filename=../fr3/meshes/visual/link7_0.stl

Commit message: Publish square-table fixed-arm training with SGS and contact termination

File: assets/urdf/fr3_xhand_description/fr3_xhand/fr3_xhand.urdf (robot description, URDF)
Before this commit: robot fr3_xhand, 39 links, 38 joints
Links:
- link fr3_link0: geometry collision mesh filename=../fr3/meshes/collision/link0.stl; visual mesh filename=../fr3/meshes/visual/link0.stl
- link fr3_link1: geometry collision mesh filename=../fr3/meshes/collision/link1.stl; visual mesh filename=../fr3/meshes/visual/link1.stl
- link fr3_link2: geometry collision mesh filename=../fr3/meshes/collision/link2.stl; visual mesh filename=../fr3/meshes/visual/link2.stl
- link fr3_link3: geometry collision mesh filename=../fr3/meshes/collision/link3.stl; visual mesh filename=../fr3/meshes/visual/link3.stl
- link fr3_link4: geometry collision mesh filename=../fr3/meshes/collision/link4.stl; visual mesh filename=../fr3/meshes/visual/link4.stl
- link fr3_link5: geometry collision mesh filename=../fr3/meshes/collision/link5.stl; visual mesh filename=../fr3/meshes/visual/link5.stl
- link fr3_link6: geometry collision mesh filename=../fr3/meshes/collision/link6.stl; visual mesh filename=../fr3/meshes/visual/link6.stl
- link fr3_link7: geometry collision mesh filename=../fr3/meshes/collision/link7.stl; visual mesh filename=../fr3/meshes/visual/link7.stl
